File: FINAL/final.brd (EAGLE design)
At the start: 151 x 113 mm, 43 parts

Commit message: Add final version files
Parts:
- R12, R22, R24, R28, R31, R7: device rcl:R0805 -> rcl:0207/15
- moved U$6 169.4 mm to (58.9, 79.9), turned to 180 degrees
- moved R9 119.2 mm to (52.0, 70.6), turned to 180 degrees
- moved R25 118.1 mm to (56.9, 58.9)
- moved R26 118.1 mm to (50.9, 55.9), turned to 180 degrees
- moved U$3 80.8 mm to (16.9, 54.9)
- moved R4 62.5 mm to (56.1, 66.9), turned to 0 degrees
- moved R6 58.9 mm to (60.9, 66.9)
- moved R34 57.8 mm to (55.8, 62.3), turned to 180 degrees
- moved R18 56.1 mm to (56.5, 70.6), turned to 180 degrees
- moved R35 54.7 mm to (64.5, 65.9), turned to 270 degrees
- moved R1 51.9 mm to (50.2, 61.9), turned to 180 degrees
- moved U$2 46.5 mm to (23.9, 20.9)
- moved R2 45.4 mm to (50.4, 59.0), turned to 180 degrees
- moved R10 39.0 mm to (13.0, 67.0), flipped to the top, turned to 90 degrees
- moved R8 38.5 mm to (25.4, 54.0), flipped to the top, turned to 90 degrees
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Connections:
- net GND: now also HILO.3, HILO.5
- net N$22: now also R31.2
- net N$23: now also R24.2
- net N$26: now also R21.2
- net N$9: now also R18.2
- net VDD: no longer HILO.3, HILO.5
Routing:
- net VCC: track 0.00 -> 159.4 mm, vias 0 -> 2
- net A_LO-HI_OUT: track 0.00 -> 119.5 mm
- net A_HI-LO_OUT: track 0.00 -> 113.2 mm
- net VDD: track 0.00 -> 110.5 mm
- net N$2: track 0.00 -> 64.2 mm
- net A_HI-LO_IN: track 0.00 -> 62.0 mm
- net A_LO-HI_IN: track 0.00 -> 52.2 mm, vias 0 -> 1
- net N$46: track 0.00 -> 52.2 mm, vias 0 -> 2
- net N$10: track 0.00 -> 51.8 mm
- net OUT1: track 0.00 -> 43.4 mm, vias 0 -> 1
- net N$18: track 0.00 -> 41.9 mm, vias 0 -> 1
- net N$42: track 0.00 -> 39.5 mm
- net N$50: track 0.00 -> 35.4 mm
- net N$4: track 0.00 -> 24.7 mm
- net N$30: track 0.00 -> 24.1 mm
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Other:
- board size 151 x 113 mm -> 73 x 108.3 mm
- board text added: "H>L_I H>L_O VDD DIGI_H DIGI_L VCC GND L>H_O L>H_I"
- board text added: "Protopaja 2016 USCO"
- board text removed: "Protopaja 13.7.2016 UADIVOLECO "Lime-Lemon""
