File: FINAL/final.sch (EAGLE design)
At the start: 43 parts

Commit message: Add final version files
Parts:
- R12, R22, R24, R28, R31, R7: device rcl:R-US_R0805 -> rcl:R-US_0207/15
Connections:
- net GND: now also HILO.1IN+, HILO.2IN+
- net N$22: now also R31.2
- net N$23: now also R24.2
- net N$26: now also R21.2
- net N$9: now also R18.2
- net VDD: no longer HILO.1IN+, HILO.2IN+
Other:
- moved on the sheet: R18
